Commit message: update models

File: rbs_assets_library/models/board/model.urdf (robot description, URDF)
Before this commit: robot board, 1 links, 0 joints
Links:
- link body: geometry collision mesh filename=board.obj scale=1.0 1.0 1.0; visual mesh filename=board.dae scale=1.0 1.0 1.0

Commit message: added new assets and added new scripts for cnos processing

File: rbs_assets_library/models/board/model.urdf (robot description, URDF)
Before this commit: robot board, 1 links, 0 joints
Links:
- removed link body
- added link board_link, mass 0.30646344250128266; collision mesh filename=board.obj scale=1.0 1.0 1.0; visual mesh filename=board.dae scale=1.0 1.0 1.0
